File: z80pc/mpu.kicad_sch (KiCad schematic)
At the start: 4 parts

Commit message: added a few net names...
Parts:
- removed U?: AS6C4008-55PIN, db-thparts:DIP-32-600MIL, symbol db-memory:AS6C4008-55PIN
- added U201: AS6C4008-55PCN, db-thparts:DIP-32-600MIL, symbol db-memory:AS6C4008-55PCN
- added U202: SST39SF040-70-4C-PHE, db-thparts:DIP-32-600MIL, symbol db-memory:SST39SF040-70-4C-PHE
- added U203: CD74HC174E, db-thparts:DIP-16-300MIL, symbol db-sem:CD74HC174E
Connections:
- net A11: now reaches U?.1 (A11)
- net A11: now also U201.25 (A11)
- net D6: now reaches U?.10 (D6)
- net D2: now reaches U?.12 (D2)
- net D2: now also U?.14 (D0)
- net D7: now reaches U?.13 (D7)
- net D1: now reaches U?.15 (D1)
- net A12: now reaches U?.2 (A12)
- net A12: now also U201.4 (A12)
- net A13: now reaches U?.3 (A13)
- net A13: now also U201.28 (A13)
- net A0: now reaches U?.30 (A0)
- net A0: now also U201.12 (A0)
- net A1: now reaches U?.31 (A1)
- net A1: now also U201.11 (A1)
- net A2: now reaches U?.32 (A2)
- net A2: now also U201.10 (A2)
- net A3: now reaches U?.33 (A3)
- net A3: now also U201.9 (A3)
- net A4: now reaches U?.34 (A4)
- net A4: now also U201.8 (A4)
- net A5: now reaches U?.35 (A5)
- net A5: now also U201.7 (A5)
- net A6: now reaches U?.36 (A6)
- net A6: now also U201.6 (A6)
- net A7: now reaches U?.37 (A7)
- net A7: now also U201.5 (A7)
- net A8: now reaches U?.38 (A8)
- net A8: now also U201.27 (A8)
- net A9: now reaches U?.39 (A9)
- net A9: now also U201.26 (A9)
- net A14: now reaches U?.4 (A14)
- net A10: now reaches U?.40 (A10)
- net A10: now also U201.23 (A10)
- net A15: now reaches U?.5 (A15)
- net D4: now reaches U?.7 (D4)
- net D3: now reaches U?.8 (D3)
- net D5: now reaches U?.9 (D5)
- new net BA0-14: U203.2 (Q0)
- new net BA0-15: U203.5 (Q1)
- new net BA0-16: U203.7 (Q2)
- new net BA0-17: U203.10 (Q3)
- new net BA0-18: U203.12 (Q4)
- new net BA0-19: U203.15 (Q5)
Other:
- note added: "RAM Bank 0"
- note added: "use 74hc153 to multiplex upper address bits in banks"
- moved on the sheet: U?, U?A, U?B

Commit message: memory mapping, etc...
Parts:
- removed U201: AS6C4008-55PCN, db-thparts:DIP-32-600MIL, symbol db-memory:AS6C4008-55PCN
- removed U202: SST39SF040-70-4C-PHE, db-thparts:DIP-32-600MIL, symbol db-memory:SST39SF040-70-4C-PHE
- removed U? (x2): SN74HC138N, db-thparts:DIP-16-300MIL, symbol db-sem:SN74HC138N
- added U203: SN74AHC139N, db-thparts:DIP-16-300MIL, symbol db-sem:SN74AHC139N
- added U204, U206, U207, U208, U? (x2): SN74HC153N, db-thparts:DIP-16-300MIL, symbol db-sem:SN74HC153N
- added U205, U?: SN74HC138N, db-thparts:DIP-16-300MIL, symbol db-sem:SN74HC138N
- added U209: SN74HC02N, db-thparts:DIP-14-300MIL, symbol db-sem:SN74HC02N
- added U?: CD74HC174E, db-thparts:DIP-16-300MIL, symbol db-sem:CD74HC174E
- added U? (x4): SN74HC574N, db-thparts:DIP-20-300MIL, symbol db-sem:SN74HC574N
- renumbered U203 to U?
Connections:
- net A0: now also U205.1 (A)
- net A1: now also U205.2 (B)
- net A14: now also U204.7 (1Y), U?.14 (A); no longer U?.4 (A14)
- net A15: now also U204.9 (2Y), U?.2 (B); no longer U?.5 (A15)
- net A2: now also U205.3 (C)
- net A4: now also U209.3 (1B)
- net A5: now also U209.2 (1A)
- net A6: now also U203.14 (2A)
- net A7: now also U203.13 (2B)
- net D1: now also U?.4 (D1), U?.3 (D1), U?.3 (D1), U?.3 (D1)
- net D2: now also U?.6 (D2), U?.3 (D0), U?.4 (D2), U?.4 (D2), U?.4 (D2); no longer U?.14 (D0)
- net D3: now also U?.11 (D3), U?.4 (D1), U?.5 (D3), U?.5 (D3), U?.5 (D3)
- net D4: now also U?.13 (D4), U?.6 (D2), U?.6 (D4), U?.6 (D4), U?.6 (D4)
- net D5: now also U?.14 (D5), U?.11 (D3), U?.7 (D5), U?.7 (D5), U?.7 (D5)
- net D6: now also U?.13 (D4), U?.8 (D6), U?.8 (D6), U?.8 (D6)
- net D7: now also U?.14 (D5), U?.9 (D7), U?.9 (D7), U?.9 (D7)
- net ~{RST}: now reaches U?.1 (~{MR})
- net ~{RST}: now also U?.1 (~{MR})
- net D0: now reaches U?.3 (D0)
- net D0: now also U?.14 (D0), U?.2 (D0), U?.2 (D0), U?.2 (D0)
- net ~{BS0_WR}: now reaches U?.9 (CP)
- net ~{BS0_WR}: now also U205.15 (Y0)
- net ~{MREQ}: now reaches U?.19 (~{MREQ})
- net ~{MREQ}: now also U?.4 (~{G2A}), U?.5 (~{G2B})
- net ~{IORQ}: now reaches U?.20 (~{IORQ})
- net ~{IORQ}: now also U203.15 (~{2G})
- net ~{RD}: now reaches U?.21 (~{RD})
- net ~{WR}: now reaches U?.22 (~{WR})
- net ~{WR}: now also U205.5 (~{G2B})
- net ~{RFSH}: now reaches U?.28 (~{RFSH})
- net ~{RFSH}: now also U?.6 (G1)
- net BA0-14 renamed BS0-14
- net BS0-14: now also U204.6 (1C0)
- net BA0-15 renamed BS0-15
- net BS0-15: now also U204.10 (2C0)
- net BA0-16 renamed BS0-16
- net BS0-16: now also U206.6 (1C0)
- net BA0-17 renamed BS0-17
- net BS0-17: now also U206.10 (2C0)
- net BA0-18 renamed BS0-18
- net BS0-18: now also U207.6 (1C0)
- net BA0-19 renamed BS0-19
- net BS0-19: now also U207.10 (2C0)
- new net: U205.6 (G1), U209.1 (1Y)
- new net A16: U206.7 (1Y)
- new net A17: U206.9 (2Y)
- new net A18: U207.7 (1Y)
- new net A19: U207.9 (2Y)
- new net A20: U208.7 (1Y)
- new net A21: U208.9 (2Y)
- new net BS1-14: U204.5 (1C1), U?.19 (Q0)
- new net BS1-15: U204.11 (2C1), U?.18 (Q1)
- new net BS1-16: U206.5 (1C1), U?.17 (Q2)
- new net BS1-17: U206.11 (2C1), U?.16 (Q3)
- new net BS1-18: U207.5 (1C1), U?.15 (Q4)
- new net BS1-19: U207.11 (2C1), U?.14 (Q5)
- new net BS1-20: U208.5 (1C1), U?.13 (Q6)
- new net BS1-21: U208.11 (2C1), U?.12 (Q7)
- new net BS2-14: U204.4 (1C2), U?.19 (Q0)
- new net BS2-15: U204.12 (2C2), U?.18 (Q1)
- new net BS2-16: U206.4 (1C2), U?.17 (Q2)
- new net BS2-17: U206.12 (2C2), U?.16 (Q3)
- new net BS2-18: U207.4 (1C2), U?.15 (Q4)
- new net BS2-19: U207.12 (2C2), U?.14 (Q5)
- new net BS2-20: U208.4 (1C2), U?.13 (Q6)
- new net BS2-21: U208.12 (2C2), U?.12 (Q7)
- new net BS3-14: U204.3 (1C3), U?.19 (Q0)
- new net BS3-15: U204.13 (2C3), U?.18 (Q1)
- new net BS3-16: U206.3 (1C3), U?.17 (Q2)
- new net BS3-17: U206.13 (2C3), U?.16 (Q3)
- new net BS3-18: U207.3 (1C3), U?.15 (Q4)
- new net BS3-19: U207.13 (2C3), U?.14 (Q5)
- new net BS3-20: U208.3 (1C3), U?.13 (Q6)
- new net BS3-21: U208.13 (2C3), U?.12 (Q7)
- new net GND: U204.1 (~{1G}), U204.15 (~{2G}), U206.1 (~{1G}), U206.15 (~{2G}), U207.1 (~{1G}), U207.15 (~{2G}), U208.1 (~{1G}), U208.10 (2C0), U208.15 (~{2G}), U208.6 (1C0), U?.1 (~{1G}), U?.10 (2C0), U?.15 (~{2G}), U?.3 (C), U?.6 (1C0)
- new net S1SS0: U?.2 (Q0), U?.5 (1C1)
- new net S1SS1: U?.11 (2C1), U?.5 (Q1)
- new net S2SS0: U?.4 (1C2), U?.7 (Q2)
- new net S2SS1: U?.10 (Q3), U?.12 (2C2)
- new net S3SS0: U?.12 (Q4), U?.3 (1C3)
- new net S3SS1: U?.13 (2C3), U?.15 (Q5)
- new net SS0: U?.1 (A), U?.7 (1Y)
- new net SS1: U?.2 (B), U?.9 (2Y)
- new net ZA14: U204.14 (A), U206.14 (A), U207.14 (A), U208.14 (A), U?.4 (A14)
- new net ZA15: U204.2 (B), U206.2 (B), U207.2 (B), U208.2 (B), U?.5 (A15)
- new net ~{BS1_WR}: U205.14 (Y1), U?.11 (CLK)
- new net ~{BS2_WR}: U205.13 (Y2), U?.11 (CLK)
- new net ~{BS3_WR}: U205.12 (Y3), U?.11 (CLK)
- new net ~{IORQ_B0}: U203.12 (2Y0), U205.4 (~{G2A})
- new net ~{IORQ_B1}: U203.11 (2Y1)
- new net ~{IORQ_B2}: U203.10 (2Y2)
- new net ~{IORQ_B3}: U203.9 (2Y3)
- new net ~{MREQ_S0}: U?.15 (Y0)
- new net ~{MREQ_S1}: U?.14 (Y1)
- new net ~{MREQ_S2}: U?.13 (Y2)
- new net ~{MREQ_S3}: U?.12 (Y3)
- new net ~{MSS_WR}: U205.11 (Y4), U?.9 (CP)
Other:
- note added: "Bank Select Registers"
- note added: "Don't clutter MREQ signals with refresh cycles"
- note added: "IO Bank 0 WR - 0x00 to 0x07"
- note added: "Memory Source Select Register"
- note removed: "RAM Bank 0"
- note removed: "use 74hc153 to multiplex upper address bits in banks"
- moved on the sheet: U?, U?A, U?B

Commit message: working
Parts:
- removed U209: SN74HC02N, db-thparts:DIP-14-300MIL, symbol db-sem:SN74HC02N
- added R201: 4.7k, db-thparts:SIP-9, symbol db-passives:4609X-101-472LF
- added U?: SN74HC574N, db-thparts:DIP-20-300MIL, symbol db-sem:SN74HC574N
- added U? (x3): SN74HC138N, db-thparts:DIP-16-300MIL, symbol db-sem:SN74HC138N
- added U? (x3): SN74HC32N, db-thparts:DIP-14-300MIL, symbol db-sem:SN74HC32N
- added U?: SN74HC02N, db-thparts:DIP-14-300MIL, symbol db-sem:SN74HC02N
- renumbered U207 to U?, U203 to U?, U206 to U?, U208 to U?, U205 to U?, U204 to U?
Connections:
- net A0: now also U?.1 (A), U?.1 (A)
- net A1: now also U?.1 (A), U?.2 (B), U?.2 (B)
- net A14: no longer U?.14 (A)
- net A15: no longer U?.2 (B)
- net A2: now also U?.2 (B), U?.3 (C), U?.3 (C)
- net A3: now also U?.3 (C)
- net A4: now also U?.3 (1B), U?.6 (G1), U?.6 (G1), U?.6 (G1)
- net A5: now also U?.1 (1A), U?.2 (1A), U?.2 (1B), U?.4 (1A)
- net D0: now also R201.9, U?.19 (Q0), U?.2 (D0)
- net D1: now also R201.8, U?.18 (Q1), U?.3 (D1)
- net D2: now also R201.7, U?.17 (Q2), U?.4 (D2)
- net D3: now also R201.6, U?.16 (Q3), U?.5 (D3)
- net D4: now also R201.5, U?.15 (Q4), U?.6 (D4)
- net D5: now also R201.4, U?.14 (Q5), U?.7 (D5)
- net D6: now also R201.3, U?.13 (Q6), U?.8 (D6)
- net D7: now also R201.2, U?.12 (Q7), U?.9 (D7)
- net GND: now also U?.1 (~{OE}), U?.1 (~{OE}), U?.1 (~{OE})
- net ZA14: now also U?.14 (A)
- net ZA15: now also U?.2 (B)
- net ~{IORQ_B0}: now also U?.4 (~{G2A}), U?.4 (~{G2A}), U?.4 (~{G2A})
- net ~{RD}: now also U?.1 (1A), U?.2 (1B)
- net ~{WR}: now also U?.5 (1B)
- net at U?.6 (G1): now also U?.1 (1Y)
- net ~{LEDS_WR}: now reaches U?.10 (Y5)
- net S1SS0 renamed S1MSS0
- net S1SS1 renamed S1MSS1
- net S2SS0 renamed S2MSS0
- net S2SS1 renamed S2MSS1
- net S3SS0 renamed S3MSS0
- net S3SS1 renamed S3MSS1
- new net: U?.3 (1Y), U?.5 (~{G2B}) (x2)
- new net: U?.5 (~{G2B}), U?.6 (1Y)
- new net ~{JOY0_RD}: U?.15 (Y0)
- new net ~{JOY1_RD}: U?.14 (Y1)
- new net ~{MEMSIZE_RD}: U?.1 (~{OE}), U?.15 (Y0)
- new net ~{MEMSIZE_WR}: U?.11 (CLK), U?.15 (Y0)
Other:
- note added: "IO Bank 0 Read-only registers Addresses 0x10 to 0x1F Mirrors on even/odd"
- note added: "IO Bank 0 Read-write registers Addresses 0x10 to 0x17"
- note added: "IO Bank 0 Write-only registers Addresses 0x00 to 0x0F 0x00-0x07 mirrored at 0x08-0x0F"
- note added: "IO Bank Chip Selects"
- note added: "Memory Source Select Register Address 0x05"
- note removed: "IO Bank 0 WR - 0x00 to 0x07"
- note removed: "Memory Source Select Register"
- moved on the sheet: U?A, U?B
