File: z80pc/z80pc.kicad_sch (KiCad schematic)
At the start: 0 parts

Commit message: memory mapping, etc...
Other:
- added sheet Memory (memory.kicad_sch)
- sheet MPU ports: added A[0..21], D[0..7], ~{MREQ_S0}, ~{MREQ_S1}, ~{MREQ_S2}, ~{MREQ_S3}, ~{RD}, ~{WR}; removed none
Changed lines of the file:
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@@
     (date "2023-10-11")
   )
-  (sheet (at 92.71 67.31) (size 13.97 29.21) (fields_autoplaced)
+  (sheet (at 77.47 59.69) (size 27.94 45.72) (fields_autoplaced)
     (stroke (width 0.1524) (type solid))
     (fill (color 0 0 0 0.0000))
-    (property "Sheetname" "MPU" (at 92.71 66.5984 0)
+    (property "Sheetname" "MPU" (at 77.47 58.9784 0)
       (effects (font (size 1.27 1.27)) (justify left bottom))
     )
-    (property "Sheetfile" "mpu.kicad_sch" (at 92.71 97.1046 0)
+    (property "Sheetfile" "mpu.kicad_sch" (at 77.47 105.9946 0)
       (effects (font (size 1.27 1.27)) (justify left top))
+    )
+    (pin "~{MREQ_S0}" output (at 105.41 69.85 0)
+      (effects (font (size 1.27 1.27)) (justify right))
+    )
+    (pin "~{MREQ_S2}" output (at 105.41 64.77 0)
+      (effects (font (size 1.27 1.27)) (justify right))
+    )
+    (pin "~{MREQ_S1}" output (at 105.41 67.31 0)
+      (effects (font (size 1.27 1.27)) (justify right))
+    )
+    (pin "~{MREQ_S3}" output (at 105.41 62.23 0)
+      (effects (font (size 1.27 1.27)) (justify right))
+    )
+    (pin "D[0..7]" bidirectional (at 105.41 82.55 0)
+      (effects (font (size 1.27 1.27)) (justify right))
+    )
+    (pin "A[0..21]" bidirectional (at 105.41 80.01 0)
+      (effects (font (size 1.27 1.27)) (justify right))
+    )
+    (pin "~{WR}" output (at 105.41 76.2 0)
+      (effects (font (size 1.27 1.27)) (justify right))
+    )
+    (pin "~{RD}" output (at 105.41 73.66 0)
+      (effects (font (size 1.27 1.27)) (justify right))
+    )
+    (instances
+      (project "z80pc"
+        (path "/153d2715-ae43-47de-9022-3a4a786cf7e2" (page "1"))
+      )
+    )
+  )
+  (sheet (at 139.7 59.69) (size 25.4 45.72) (fields_autoplaced)
+    (stroke (width 0.1524) (type solid))
+    (fill (color 0 0 0 0.0000))
+    (property "Sheetname" "Memory" (at 139.7 58.9784 0)
+      (effects (font (size 1.27 1.27)) (justify left bottom))
+    )
+    (property "Sheetfile" "memory.kicad_sch" (at 139.7 105.9946 0)
+      (effects (font (size 1.27 1.27)) (justify left top))
+    )
+    (pin "~{MREQ}" input (at 139.7 62.23 180)
+      (effects (font (size 1.27 1.27)) (justify left))
+    )
+    (pin "A[0..21]" input (at 139.7 80.01 180)
+      (effects (font (size 1.27 1.27)) (justify left))
+    )
+    (pin "D[0..7]" bidirectional (at 139.7 82.55 180)
+      (effects (font (size 1.27 1.27)) (justify left))
     )
     (instances
@@
   )
   (sheet_instances
-    (path "/" (page "1"))
+    (path "/" (page "0"))
   )
 )

Commit message: working
Other:
- added sheet IO Ports (ioports.kicad_sch)
- sheet MPU ports: added ~{IORQ_B0}, ~{IORQ_B1}, ~{IORQ_B2}, ~{IORQ_B3}, ~{JOY0_RD}, ~{JOY1_RD}; removed none
Changed lines of the file:
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@@
     (date "2023-10-11")
   )
-  (sheet (at 77.47 59.69) (size 27.94 45.72) (fields_autoplaced)
+  (sheet (at 77.47 59.69) (size 27.94 59.69) (fields_autoplaced)
     (stroke (width 0.1524) (type solid))
     (fill (color 0 0 0 0.0000))
@@
       (effects (font (size 1.27 1.27)) (justify left bottom))
     )
-    (property "Sheetfile" "mpu.kicad_sch" (at 77.47 105.9946 0)
+    (property "Sheetfile" "mpu.kicad_sch" (at 77.47 119.9646 0)
       (effects (font (size 1.27 1.27)) (justify left top))
     )
@@
       (effects (font (size 1.27 1.27)) (justify right))
     )
-    (pin "D[0..7]" bidirectional (at 105.41 82.55 0)
+    (pin "D[0..7]" bidirectional (at 105.41 113.03 0)
       (effects (font (size 1.27 1.27)) (justify right))
     )
-    (pin "A[0..21]" bidirectional (at 105.41 80.01 0)
+    (pin "A[0..21]" bidirectional (at 105.41 110.49 0)
       (effects (font (size 1.27 1.27)) (justify right))
     )
-    (pin "~{WR}" output (at 105.41 76.2 0)
+    (pin "~{WR}" output (at 105.41 104.14 0)
       (effects (font (size 1.27 1.27)) (justify right))
     )
-    (pin "~{RD}" output (at 105.41 73.66 0)
+    (pin "~{RD}" output (at 105.41 101.6 0)
+      (effects (font (size 1.27 1.27)) (justify right))
+    )
+    (pin "~{IORQ_B0}" output (at 105.41 83.82 0)
+      (effects (font (size 1.27 1.27)) (justify right))
+    )
+    (pin "~{IORQ_B2}" output (at 105.41 78.74 0)
+      (effects (font (size 1.27 1.27)) (justify right))
+    )
+    (pin "~{IORQ_B1}" output (at 105.41 81.28 0)
+      (effects (font (size 1.27 1.27)) (justify right))
+    )
+    (pin "~{IORQ_B3}" output (at 105.41 76.2 0)
+      (effects (font (size 1.27 1.27)) (justify right))
+    )
+    (pin "~{JOY1_RD}" output (at 105.41 88.9 0)
+      (effects (font (size 1.27 1.27)) (justify right))
+    )
+    (pin "~{JOY0_RD}" output (at 105.41 91.44 0)
       (effects (font (size 1.27 1.27)) (justify right))
     )
     (instances
       (project "z80pc"
-        (path "/153d2715-ae43-47de-9022-3a4a786cf7e2" (page "1"))
+        (path "/153d2715-ae43-47de-9022-3a4a786cf7e2" (page "2"))
       )
     )
@@
     (instances
       (project "z80pc"
-        (path "/153d2715-ae43-47de-9022-3a4a786cf7e2" (page "2"))
+        (path "/153d2715-ae43-47de-9022-3a4a786cf7e2" (page "3"))
+      )
+    )
+  )
+  (sheet (at 139.7 119.38) (size 25.4 39.37) (fields_autoplaced)
+    (stroke (width 0.1524) (type solid))
+    (fill (color 0 0 0 0.0000))
+    (property "Sheetname" "IO Ports" (at 139.7 118.6684 0)
+      (effects (font (size 1.27 1.27)) (justify left bottom))
+    )
+    (property "Sheetfile" "ioports.kicad_sch" (at 139.7 159.3346 0)
+      (effects (font (size 1.27 1.27)) (justify left top))
+    )
+    (instances
+      (project "z80pc"
+        (path "/153d2715-ae43-47de-9022-3a4a786cf7e2" (page "4"))
       )
     )
   )
   (sheet_instances
-    (path "/" (page "0"))
+    (path "/" (page "1"))
   )
 )
